File: Tarjeta de presentación/Tarjeta_present.sch (KiCad schematic (older format))
At the start: 11 parts, among them J1 Conn_01x01_Female, J2 USB_A, SW1 Reset, SW2 Boot, U1 CH552G

Commit message: Add ground template
Parts:
- U1: symbol Librerias:CH552G -> Tarjeta_present-rescue:CH552G-Librerias
Changed lines of the file:
@@
 $EndDescr
 $Comp
-L Librerias:CH552G U1
+L Tarjeta_present-rescue:CH552G-Librerias U1
 U 1 1 600C5722
 P 4350 2650
