File: hardware/card_business.kicad_pcb (KiCad board)
At the start: 2 copper layers, 49.9 x 17.3 mm, 11 parts, among them J1 Conn_01x01_Female, J2 USB_A, SW1 Reset, SW2 Boot, U1 CH552G

Commit message: routing complete
Parts:
- moved U1 0.62 mm to (114.6, 83.7)
Routing:
- net /PAD: track 11.2 -> 12.5 mm
- net GND: track 32.4 -> 33.7 mm
- net /P3.3: track 13.4 -> 14.6 mm
- net /UDM: track 25.7 -> 26.9 mm
- net +5V: track 43.9 -> 44.9 mm
- net /RST: track 3.66 -> 4.41 mm

Commit message: add labels and logo
Parts:
- added G***: LOGO, Aesthetics:electronic_cats_logo_4x3, F.Cu at (128.0, 99.8)
Routing:
- added copper zone on B.Cu, net GND
- removed copper zone on B.Cu, net (none)
Other:
- board text added: "Andrés Sabas"
- board text added: "Phone: XXXXXXXXXX"

Commit message: side change
Parts:
- C1, C2, D1, R1, R2, R3, U1: moved to B.Cu
- moved R1 14.6 mm to (110.1, 77.7), turned to 0 degrees
- moved R3 12.9 mm to (111.6, 91.3), turned to 0 degrees
- moved D1 12.5 mm to (107.5, 91.3), turned to 0 degrees
- moved SW1 11.3 mm to (116.8, 82.4), turned to 90 degrees
- moved G*** 10.2 mm to (126.5, 89.7)
- moved SW2 8.82 mm to (123.9, 77.9)
- moved R2 6.29 mm to (116.8, 87.2), turned to 270 degrees
- moved C1 5.34 mm to (102.2, 90.2), turned to 90 degrees
- moved U1 5.26 mm to (109.4, 84.5), turned to 270 degrees
- moved J1 2.03 mm to (131.1, 79.7)
- moved C2 0.25 mm to (102.1, 86.1), turned to 180 degrees
Routing:
- net Net-(R2-Pad1): track 2.04 -> 15.7 mm, vias 0 -> 1
- net /PAD: track 12.5 -> 23.7 mm, vias 0 -> 1
- net /P3.3: track 14.6 -> 3.58 mm
- net +5V: track 44.9 -> 53.7 mm, vias 0 -> 1
- net /UDM: track 26.9 -> 20.4 mm, vias 2 -> 1
- net GND: track 33.7 -> 28.1 mm, vias 0 -> 1
- net Net-(R1-Pad2): track 2.03 -> 7.22 mm, vias 0 -> 1
- net /UDP: track 36.0 -> 32.0 mm, vias 2 -> 1
- net Net-(D1-Pad2): track 3.99 -> 2.24 mm
- net /RST: track 4.41 -> 5.17 mm

Commit message: labels
Parts:
- moved G*** 20.4 mm to (108.2, 80.7)
- renumbered SW2 to BOOT, SW1 to RST

Commit message: change routing
Parts:
- D1: moved to F.Cu
- moved G*** 24.1 mm to (132.4, 79.7)
- moved SW2 15.1 mm to (118.9, 92.2), turned to 90 degrees
- moved SW1 10.6 mm to (125.9, 87.8), turned to 270 degrees
- moved R1 10.4 mm to (116.6, 85.9)
- moved J1 10.2 mm to (131.9, 89.8)
- moved C1 8.00 mm to (101.3, 82.3), turned to 0 degrees
- moved C2 7.13 mm to (101.3, 79.0), turned to 0 degrees
- moved R2 5.27 mm to (114.0, 91.6), turned to 180 degrees
- moved D1 3.84 mm to (103.7, 91.5)
- moved R3 1.72 mm to (109.9, 91.6)
- moved U1 0.96 mm to (110.2, 84.0), turned to 180 degrees
- moved J2 0.08 mm to (86.4, 84.9)
- renumbered RST to SW1, BOOT to SW2
Connections:
- U1 pad 2: Net-(U1-Pad2) -> /PAD
- U1 pad 9: /PAD -> Net-(U1-Pad9)
Routing:
- net GND: track 28.1 -> 43.6 mm, vias 1 -> 2
- net Net-(R2-Pad1): track 15.7 -> 8.59 mm
- net Net-(R1-Pad2): track 7.22 -> 12.2 mm
- net +5V: track 53.7 -> 49.0 mm, vias 1 -> 2
- net /UDM: track 20.4 -> 24.9 mm
- net /P3.3: track 3.58 -> 7.75 mm
- net /UDP: track 32.0 -> 28.0 mm, vias 1 -> 3
- net /PAD: track 23.7 -> 27.0 mm
- net Net-(D1-Pad2): track 2.24 -> 5.20 mm, vias 0 -> 1
- net /RST: track 5.17 -> 2.25 mm

Commit message: routing update
Routing:
- net +5V: track 49.0 -> 49.8 mm
